File: USB-HW/USB-HW.kicad_pcb (KiCad board)
At the start: 2 copper layers, 0 parts

Commit message: feat: Add PCB
Parts:
- added C1: 10n, Capacitor_SMD:C_0805_2012Metric, F.Cu at (125.5, 75.0)
- added C2: 100n, Capacitor_SMD:C_0805_2012Metric, F.Cu at (125.5, 68.0)
- added C3: 4u7, Capacitor_SMD:CP_Elec_4x5.3, F.Cu at (126.0, 42.3)
- added C4: 100n, Capacitor_SMD:C_0805_2012Metric, F.Cu at (120.3, 69.2)
- added C5: 4u7, Capacitor_SMD:CP_Elec_4x5.3, F.Cu at (104.5, 42.5)
- added C6: 100n, Capacitor_SMD:C_0805_2012Metric, F.Cu at (120.3, 65.5)
- added C7: 1u, Capacitor_SMD:C_0805_2012Metric, F.Cu at (125.5, 64.8)
- added FB1: 100, Inductor_SMD:L_0805_2012Metric, F.Cu at (125.6, 71.5)
- added H1: UART Interface, Connector_PinHeader_2.54mm:PinHeader_1x05_P2.54mm_Vertical, F.Cu at (110.1, 41.8)
- added H2: RS-232 Interface, Connector_PinSocket_2.54mm:PinSocket_1x06_P2.54mm_Vertical, F.Cu at (108.9, 57.0)
- added J1: USB A, Connector_USB:USB_A_Molex_48037-2200_Horizontal, F.Cu at (115.0, 83.5)
- added LD1: LED RX, LED_SMD:LED_0805_2012Metric, F.Cu at (110.2, 47.3)
- added LD2: LED TX, LED_SMD:LED_0805_2012Metric, F.Cu at (113.5, 47.3)
- added LD3: LED 5V, LED_SMD:LED_0805_2012Metric, F.Cu at (116.8, 47.3)
- added LD4: LED 3V3, LED_SMD:LED_0805_2012Metric, F.Cu at (119.8, 47.3)
- added R1: 330, Resistor_SMD:R_0805_2012Metric, F.Cu at (110.2, 51.7)
- added R2: 330, Resistor_SMD:R_0805_2012Metric, F.Cu at (113.5, 51.7)
- added R3: 330, Resistor_SMD:R_0805_2012Metric, F.Cu at (116.8, 51.7)
- added R4: 120, Resistor_SMD:R_0805_2012Metric, F.Cu at (119.8, 51.7)
- added U1: SP0503BAHTG, Package_TO_SOT_SMD:SOT-143, F.Cu at (105.0, 73.5)
- added U2: CP2102, Package_DFN_QFN:QFN-28-1EP_5x5mm_P0.5mm_EP3.25x3.25mm, F.Cu at (114.8, 63.9)
Routing:
- net +3V3: track 0.00 -> 93.2 mm, vias 0 -> 3
- net +5V: track 0.00 -> 67.3 mm
- net TX: track 0.00 -> 42.0 mm, vias 0 -> 2
- net VBUS: track 0.00 -> 32.6 mm, vias 0 -> 2
- net RX: track 0.00 -> 30.9 mm, vias 0 -> 2
- net D_P: track 0.00 -> 25.4 mm, vias 0 -> 2
- net D_N: track 0.00 -> 23.0 mm, vias 0 -> 2
- net RI: track 0.00 -> 15.2 mm, vias 0 -> 1
- net DCD: track 0.00 -> 14.8 mm, vias 0 -> 1
- net DTR: track 0.00 -> 14.2 mm
- net DSR: track 0.00 -> 12.9 mm
- net CTS: track 0.00 -> 11.0 mm
- net RTS: track 0.00 -> 9.05 mm
- net Net-(LD4-A): track 0.00 -> 2.50 mm
- net Net-(LD3-A): track 0.00 -> 2.50 mm
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- added copper zone on F.Cu, net GND
Other:
- board outline added: 30 x 40 mm
- board text added: "3V3"
- board text added: "5V"
- board text added: "GND"
- board text added: "RX"
- board text added: "TX"
- board text added: "USB-HW"
